Commit message: fix: URDF 限速统一 + place 前置夹持检查
## URDF 限速
6 个臂关节是 velocity="1"（57°/s），两个夹爪关节是 3.14（180°/s）；
而 joint_limits.yaml 的 max_velocity: 3.14 会覆盖 URDF。
也就是说 URDF 里那个 1 从未生效，但看 URDF 的人会以为限速是 57°/s。

统一为 3.14，与 yaml 一致、与真机已跑通 13 次的配置一致。
⚠ cello_description 在 install 里是**拷贝**，改 URDF 必须 colcon build 才生效
（已验证 install 里现在是 8 个 3.14、0 个 1）。

## place 前置检查
--phase place 之前读 joint7_left 判断手上有没有东西：

| 开口 | 判定 |
|---|---|
| ≤ 9.5 mm（合到底） | 没东西 |
| ≥ 64 mm（全开） | 没东西（上一轮 pick 失败会停在这） |
| 中间 | 视为夹着，继续 |

空放不仅白跑一趟，还可能把夹爪怼到台面上。`--no-grasp-check` 可跳过。

⚠ 判据的边界：夹爪最小开口就是 8 mm（结构间隙），比它薄的物体本来也夹不住，
这套判据对那种情况无从分辨。

dry-run 不连硬件，自动跳过检查。

File: star-arm-moveit2/src/cello_description/urdf/cello_description.urdf (robot description, URDF)
Before this commit: robot cello_description, 10 links, 9 joints
Joints:
- joint joint1: limit lower=-2.27 upper=2.27 effort=100 velocity=1 -> lower=-2.27 upper=2.27 effort=100 velocity=3.14
- joint joint2: limit lower=-1.57 upper=1.57 effort=100 velocity=1 -> lower=-1.57 upper=1.57 effort=100 velocity=3.14
- joint joint3: limit lower=-1.57 upper=1.57 effort=100 velocity=1 -> lower=-1.57 upper=1.57 effort=100 velocity=3.14
- joint joint4: limit lower=-2.27 upper=2.27 effort=100 velocity=1 -> lower=-2.27 upper=2.27 effort=100 velocity=3.14
- joint joint5: limit lower=-1.57 upper=1.57 effort=100 velocity=1 -> lower=-1.57 upper=1.57 effort=100 velocity=3.14
- joint joint6: limit lower=-2.27 upper=2.27 effort=100 velocity=1 -> lower=-2.27 upper=2.27 effort=100 velocity=3.14
